File: hardware/EVNotipi-RasPi-Watchdog-Adapter/EVNotipi-RasPi-Watchdog-Adapter.kicad_pcb (KiCad board)
At the start: 2 copper layers, 10.8 x 50.8 mm, 2 parts, among them J1 Conn_Pi, J2 Raspberry_Pi_2_3

Commit message: Add labels to silk scren
Parts:
- moved J1 1054.6 mm to (31.8, 27.9)
- moved J2 1054.6 mm to (29.2, 20.2)
Other:
- board size 10.8 x 50.8 mm -> 11.4 x 50.8 mm
- board text added: "GND"
- board text added: "RUN"
- board text added: "SCL"
- board text added: "SDA"
- board text added: "VCC"
Changed lines of the file:
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@@
   (general
     (thickness 1.6)
-    (drawings 8)
+    (drawings 13)
     (tracks 33)
     (zones 0)
@@
   )
   (module Connector_PinHeader_2.54mm:PinHeader_1x05_P2.54mm_Horizontal (layer F.Cu)
-    (at 1082.675 -60.325)
+    (at 31.75 27.94)
     (descr "Through hole angled pin header, 1x05, 2.54mm pitch, 6mm pin length, single row")
     (tags "Through hole angled pin header THT 1x05 2.54mm single row")
-    (fp_text reference J1 (at 4.385 -2.27) (layer F.SilkS)
+    (fp_text reference J1 (at 0.635 -2.54) (layer F.SilkS)
       (effects (font (size 1 1) (thickness 0.15)))
     )
@@
   )
   (module Connector_PinSocket_2.54mm:PinSocket_2x20_P2.54mm_Vertical (layer F.Cu)
-    (at 1080.135 -68.024999)
+    (at 29.21 20.240001)
     (descr "Through hole straight socket strip, 2x20, 2.54mm pitch, double cols (from Kicad 4.0.7), script generated")
     (tags "Through hole socket strip THT 2x20 2.54mm double row")
-    (fp_text reference J2 (at -1.27 -2.77) (layer F.SilkS)
+    (fp_text reference J2 (at 2.54 21.669999 -90) (layer F.SilkS)
       (effects (font (size 1 1) (thickness 0.15)))
     )
@@
     )
   )
-  (gr_line (start 1082.04 -69.215) (end 1082.04 -65.405) (layer Edge.Cuts) (width 0.1))
-  (gr_line (start 1075.69 -69.215) (end 1082.04 -69.215) (layer Edge.Cuts) (width 0.1))
-  (gr_line (start 1075.69 -18.415) (end 1075.69 -69.215) (layer Edge.Cuts) (width 0.1))
-  (gr_line (start 1082.04 -18.415) (end 1075.69 -18.415) (layer Edge.Cuts) (width 0.1))
-  (gr_line (start 1082.04 -43.815) (end 1082.04 -18.415) (layer Edge.Cuts) (width 0.1))
-  (gr_line (start 1086.485 -48.26) (end 1082.04 -43.815) (layer Edge.Cuts) (width 0.1))
-  (gr_line (start 1086.485 -61.595) (end 1086.485 -48.26) (layer Edge.Cuts) (width 0.1))
-  (gr_line (start 1082.04 -65.405) (end 1086.485 -61.595) (layer Edge.Cuts) (width 0.1))
-  (segment (start 1083.775 -60.325) (end 1082.675 -60.325) (width 0.25) (layer B.Cu) (net 1))
-  (segment (start 1083.850001 -60.249999) (end 1083.775 -60.325) (width 0.25) (layer B.Cu) (net 1))
-  (segment (start 1081.310001 -23.48) (end 1081.310001 -46.99) (width 0.25) (layer B.Cu) (net 1))
-  (segment (start 1081.310001 -46.99) (end 1081.945001 -47.530001) (width 0.25) (layer B.Cu) (net 1))
-  (segment (start 1080.135 -22.304999) (end 1081.310001 -23.48) (width 0.25) (layer B.Cu) (net 1))
-  (segment (start 1081.945001 -47.530001) (end 1083.945 -49.53) (width 0.25) (layer B.Cu) (net 1))
-  (segment (start 1083.945 -49.53) (end 1083.850001 -60.249999) (width 0.25) (layer B.Cu) (net 1))
-  (segment (start 1080.984999 -64.635) (end 1080.135 -65.484999) (width 0.25) (layer B.Cu) (net 2))
-  (segment (start 1081.499999 -58.960001) (end 1081.499999 -64.12) (width 0.25) (layer B.Cu) (net 2))
-  (segment (start 1081.499999 -64.12) (end 1080.984999 -64.635) (width 0.25) (layer B.Cu) (net 2))
-  (segment (start 1082.675 -57.785) (end 1081.499999 -58.960001) (width 0.25) (layer B.Cu) (net 2))
-  (segment (start 1080.984999 -62.095) (end 1080.135 -62.944999) (width 0.25) (layer F.Cu) (net 3))
-  (segment (start 1081.405 -61.674999) (end 1080.984999 -62.095) (width 0.25) (layer F.Cu) (net 3))
-  (segment (start 1081.405 -57.315998) (end 1081.405 -61.674999) (width 0.25) (layer F.Cu) (net 3))
-  (segment (start 1082.675 -56.045998) (end 1081.405 -57.315998) (width 0.25) (layer F.Cu) (net 3))
-  (segment (start 1082.675 -55.245) (end 1082.675 -56.045998) (width 0.25) (layer F.Cu) (net 3))
-  (segment (start 1078.770001 -64.309998) (end 1078.444999 -64.635) (width 0.25) (layer B.Cu) (net 4))
-  (segment (start 1078.770001 -57.490996) (end 1078.770001 -64.309998) (width 0.25) (layer B.Cu) (net 4))
-  (segment (start 1079.570999 -56.689998) (end 1078.770001 -57.490996) (width 0.25) (layer B.Cu) (net 4))
-  (segment (start 1078.444999 -64.635) (end 1077.595 -65.484999) (width 0.25) (layer B.Cu) (net 4))
-  (segment (start 1080.509003 -56.689998) (end 1079.570999 -56.689998) (width 0.25) (layer B.Cu) (net 4))
-  (segment (start 1081.310001 -55.889) (end 1080.509003 -56.689998) (width 0.25) (layer B.Cu) (net 4))
-  (segment (start 1081.310001 -54.069999) (end 1081.310001 -55.889) (width 0.25) (layer B.Cu) (net 4))
-  (segment (start 1082.675 -52.705) (end 1081.310001 -54.069999) (width 0.25) (layer B.Cu) (net 4))
-  (segment (start 1078.444999 -62.095) (end 1077.595 -62.944999) (width 0.25) (layer F.Cu) (net 5))
-  (segment (start 1078.770001 -57.490996) (end 1078.770001 -61.769998) (width 0.25) (layer F.Cu) (net 5))
-  (segment (start 1079.570999 -56.689998) (end 1078.770001 -57.490996) (width 0.25) (layer F.Cu) (net 5))
-  (segment (start 1080.509003 -56.689998) (end 1079.570999 -56.689998) (width 0.25) (layer F.Cu) (net 5))
-  (segment (start 1081.405 -55.794001) (end 1080.509003 -56.689998) (width 0.25) (layer F.Cu) (net 5))
-  (segment (start 1078.770001 -61.769998) (end 1078.444999 -62.095) (width 0.25) (layer F.Cu) (net 5))
-  (segment (start 1081.405 -52.235998) (end 1081.405 -55.794001) (width 0.25) (layer F.Cu) (net 5))
-  (segment (start 1082.675 -50.965998) (end 1081.405 -52.235998) (width 0.25) (layer F.Cu) (net 5))
-  (segment (start 1082.675 -50.165) (end 1082.675 -50.965998) (width 0.25) (layer F.Cu) (net 5))
+  (gr_text RUN (at 34.29 27.94 180) (layer B.SilkS)
+    (effects (font (size 1 1) (thickness 0.15)) (justify mirror))
+  )
+  (gr_text GND (at 34.29 38.1 180) (layer B.SilkS)
+    (effects (font (size 1 1) (thickness 0.15)) (justify mirror))
+  )
+  (gr_text VCC (at 34.29 35.56 180) (layer B.SilkS)
+    (effects (font (size 1 1) (thickness 0.15)) (justify mirror))
+  )
+  (gr_text SCL (at 34.29 33.02 180) (layer B.SilkS)
+    (effects (font (size 1 1) (thickness 0.15)) (justify mirror))
+  )
+  (gr_text SDA (at 34.29 30.48 180) (layer B.SilkS)
+    (effects (font (size 1 1) (thickness 0.15)) (justify mirror))
+  )
+  (gr_line (start 31.115 19.05) (end 31.115 21.59) (layer Edge.Cuts) (width 0.1))
+  (gr_line (start 24.765 19.05) (end 31.115 19.05) (layer Edge.Cuts) (width 0.1))
+  (gr_line (start 24.765 69.85) (end 24.765 19.05) (layer Edge.Cuts) (width 0.1))
+  (gr_line (start 31.115 69.85) (end 24.765 69.85) (layer Edge.Cuts) (width 0.1))
+  (gr_line (start 31.115 44.45) (end 31.115 69.85) (layer Edge.Cuts) (width 0.1))
+  (gr_line (start 36.195 39.37) (end 31.115 44.45) (layer Edge.Cuts) (width 0.1))
+  (gr_line (start 36.195 26.67) (end 36.195 39.37) (layer Edge.Cuts) (width 0.1))
+  (gr_line (start 31.115 21.59) (end 36.195 26.67) (layer Edge.Cuts) (width 0.1))
+  (segment (start 32.85 27.94) (end 31.75 27.94) (width 0.25) (layer B.Cu) (net 1))
+  (segment (start 32.925001 28.015001) (end 32.85 27.94) (width 0.25) (layer B.Cu) (net 1))
+  (segment (start 30.385001 64.785) (end 30.385001 41.275) (width 0.25) (layer B.Cu) (net 1))
+  (segment (start 30.385001 41.275) (end 31.020001 40.734999) (width 0.25) (layer B.Cu) (net 1))
+  (segment (start 29.21 65.960001) (end 30.385001 64.785) (width 0.25) (layer B.Cu) (net 1))
+  (segment (start 31.020001 40.734999) (end 33.02 38.735) (width 0.25) (layer B.Cu) (net 1))
+  (segment (start 33.02 38.735) (end 32.925001 28.015001) (width 0.25) (layer B.Cu) (net 1))
+  (segment (start 30.059999 23.63) (end 29.21 22.780001) (width 0.25) (layer B.Cu) (net 2))
+  (segment (start 30.574999 29.304999) (end 30.574999 24.145) (width 0.25) (layer B.Cu) (net 2))
+  (segment (start 30.574999 24.145) (end 30.059999 23.63) (width 0.25) (layer B.Cu) (net 2))
+  (segment (start 31.75 30.48) (end 30.574999 29.304999) (width 0.25) (layer B.Cu) (net 2))
+  (segment (start 30.059999 26.17) (end 29.21 25.320001) (width 0.25) (layer F.Cu) (net 3))
+  (segment (start 30.48 26.590001) (end 30.059999 26.17) (width 0.25) (layer F.Cu) (net 3))
+  (segment (start 30.48 30.949002) (end 30.48 26.590001) (width 0.25) (layer F.Cu) (net 3))
+  (segment (start 31.75 32.219002) (end 30.48 30.949002) (width 0.25) (layer F.Cu) (net 3))
+  (segment (start 31.75 33.02) (end 31.75 32.219002) (width 0.25) (layer F.Cu) (net 3))
+  (segment (start 27.845001 23.955002) (end 27.519999 23.63) (width 0.25) (layer B.Cu) (net 4))
+  (segment (start 27.845001 30.774004) (end 27.845001 23.955002) (width 0.25) (layer B.Cu) (net 4))
+  (segment (start 28.645999 31.575002) (end 27.845001 30.774004) (width 0.25) (layer B.Cu) (net 4))
+  (segment (start 27.519999 23.63) (end 26.67 22.780001) (width 0.25) (layer B.Cu) (net 4))
+  (segment (start 29.584003 31.575002) (end 28.645999 31.575002) (width 0.25) (layer B.Cu) (net 4))
+  (segment (start 30.385001 32.376) (end 29.584003 31.575002) (width 0.25) (layer B.Cu) (net 4))
+  (segment (start 30.385001 34.195001) (end 30.385001 32.376) (width 0.25) (layer B.Cu) (net 4))
+  (segment (start 31.75 35.56) (end 30.385001 34.195001) (width 0.25) (layer B.Cu) (net 4))
+  (segment (start 27.519999 26.17) (end 26.67 25.320001) (width 0.25) (layer F.Cu) (net 5))
+  (segment (start 27.845001 30.774004) (end 27.845001 26.495002) (width 0.25) (layer F.Cu) (net 5))
+  (segment (start 28.645999 31.575002) (end 27.845001 30.774004) (width 0.25) (layer F.Cu) (net 5))
+  (segment (start 29.584003 31.575002) (end 28.645999 31.575002) (width 0.25) (layer F.Cu) (net 5))
+  (segment (start 30.48 32.470999) (end 29.584003 31.575002) (width 0.25) (layer F.Cu) (net 5))
+  (segment (start 27.845001 26.495002) (end 27.519999 26.17) (width 0.25) (layer F.Cu) (net 5))
+  (segment (start 30.48 36.029002) (end 30.48 32.470999) (width 0.25) (layer F.Cu) (net 5))
+  (segment (start 31.75 37.299002) (end 30.48 36.029002) (width 0.25) (layer F.Cu) (net 5))
+  (segment (start 31.75 38.1) (end 31.75 37.299002) (width 0.25) (layer F.Cu) (net 5))
 )
